File: projects/OBC/obc.sch (EAGLE design)
At the start: 78 parts, among them Q1 FA-128, U1 MIMXRT1052DVL6A

Commit message: Add files via upload
Parts:
- removed C55, C56: 1uF, rcl:C-EUC0402K
- removed TP4: TPTP06R, testpad:TPTP06R
- added IC1: IS42S16160J-6BLI, SDRAM_and_HyperFlash:IS42S16160J-6BLI
- added IC2: S26KS512SDPBHI020, SDRAM_and_HyperFlash:S26KS512SDPBHI020
- added R13: 0 Ohm, rcl:R-EU_R0402
- added R14, R15: 100K Ohm, rcl:R-EU_R0402
Connections:
- removed net 5V_USB_HS: C56.1, U1.USB_OTG2_VBUS
- removed net 5V_USB_OTG: C55.1, U1.USB_OTG1_VBUS
- removed net OTG1_DN: U1.USB_OTG1_DN
- removed net OTG1_DP: U1.USB_OTG1_DP
- removed net OTG2_DN: U1.USB_OTG2_DN
- removed net OTG2_DP: U1.USB_OTG2_DP
- new net N$12: IC1.CKE, R14.2
- new net N$14: IC1.DQMH
- new net N$15: IC1.DQML
- new net N$16: IC1.!CS, R15.1
- new net N$17: R15.2
- new net N$18: IC1.!WE
- new net N$19: IC1.!RAS
- new net N$20: IC1.!CAS
- new net N$21: IC1.BA1
- new net N$22: IC1.BA0
- new net N$23: R13.1
- new net N$24: IC1.VDD_3
- new net N$25: IC1.VDD_2
- new net N$28: IC1.VDDQ_1, IC1.VDDQ_2, IC1.VDDQ_3, IC1.VDDQ_4, IC1.VDD_1
- net GND: now also IC1.VSSQ_1, IC1.VSSQ_2, IC1.VSSQ_3, IC1.VSSQ_4, IC1.VSS_1, IC1.VSS_2, IC1.VSS_3, R14.1; no longer C55.2, C56.2
- net N$13: now also IC1.CLK, R13.2; no longer TP4.TP, U1.USB_OTG1_CHD_B
- net SEMC_A0: now also IC1.A0
- net SEMC_A1: now also IC1.A1
- net SEMC_A10: now also IC1.A10
- net SEMC_A11: now also IC1.A11
- net SEMC_A12: now also IC1.A12
- net SEMC_A2: now also IC1.A2
- net SEMC_A3: now also IC1.A3
- net SEMC_A4: now also IC1.A4
- net SEMC_A5: now also IC1.A5
- net SEMC_A6: now also IC1.A6
- net SEMC_A7: now also IC1.A7
- net SEMC_A8: now also IC1.A8
- net SEMC_A9: now also IC1.A9
- net SEMC_D0: now also IC1.DQ0
- net SEMC_D1: now also IC1.DQ1
- net SEMC_D10: now also IC1.DQ10
- net SEMC_D11: now also IC1.DQ11
- net SEMC_D12: now also IC1.DQ12
- net SEMC_D13: now also IC1.DQ13
- net SEMC_D14: now also IC1.DQ14
- net SEMC_D15: now also IC1.DQ15
- net SEMC_D2: now also IC1.DQ2
- net SEMC_D3: now also IC1.DQ3
- net SEMC_D4: now also IC1.DQ4
- net SEMC_D5: now also IC1.DQ5
- net SEMC_D6: now also IC1.DQ6
- net SEMC_D7: now also IC1.DQ7
- net SEMC_D8: now also IC1.DQ8
- net SEMC_D9: now also IC1.DQ9
Other:
- moved on the sheet: C1, C10, C11, C12, C13, C14, C15, C16, C17, C18, C19, C2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
